Commit message: PR06: reproduce misplaced lidar by attaching it to camera_link

File: src/course_description/urdf/vehicle.urdf.xacro (robot description, xacro)
@@ -153,5 +153,5 @@
   </link>
   <joint name="lidar_joint" type="fixed">
-    <parent link="base_link"/><child link="lidar_link"/>
+    <parent link="camera_link"/><child link="lidar_link"/>
     <origin xyz="0.28 0 0.38"/>
   </joint>

Commit message: PR06: restore lidar parent and add required checks and demonstration

File: src/course_description/urdf/vehicle.urdf.xacro (robot description, xacro)
@@ -153,5 +153,5 @@
   </link>
   <joint name="lidar_joint" type="fixed">
-    <parent link="camera_link"/><child link="lidar_link"/>
+    <parent link="base_link"/><child link="lidar_link"/>
     <origin xyz="0.28 0 0.38"/>
   </joint>
